Commit message: oops i forgot to push

File: src/climber_base/urdf/climber_robot.urdf.xacro (robot description, xacro)
@@ -7,5 +7,5 @@
   <!-- The robot wraps around a cylinder and climbs it -->
   <!-- Cylinder dimensions (the pole being climbed) -->
-  <xacro:property name="cylinder_diameter" value="0.15"/>  <!-- 15cm diameter pole -->
+  <xacro:property name="cylinder_diameter" value=".40"/>  <!-- 30cm diameter pole -->
   <xacro:property name="cylinder_radius" value="${cylinder_diameter/2}"/>
   <!-- Mecanum wheel properties -->
@@ -17,8 +17,8 @@
   <xacro:property name="wheel_radial_distance" value="${cylinder_radius + wheel_width/2}"/>
   <!-- Linear actuator properties -->
-  <xacro:property name="actuator_stroke" value="0.05"/>       <!-- 5cm total travel -->
+  <xacro:property name="actuator_stroke" value="0.16"/>       <!-- 16cm total travel -->
   <xacro:property name="actuator_home" value="0.0"/>          <!-- 0 = wheel touching cylinder -->
   <xacro:property name="actuator_min" value="-0.01"/>         <!-- 1cm inward (pressing into cylinder) -->
-  <xacro:property name="actuator_max" value="${actuator_stroke - 0.01}"/>  <!-- 4cm outward (releasing) -->
+  <xacro:property name="actuator_max" value="${actuator_stroke - 0.01}"/>  <!-- 15cm outward (releasing) -->
   <xacro:property name="actuator_mass" value="0.3"/>
   <xacro:property name="actuator_length" value="0.06"/>       <!-- Visual length of actuator body -->
@@ -27,12 +27,13 @@
   <xacro:property name="arm_length" value="0.08"/>             <!-- Radial arm from wheel outward -->
   <xacro:property name="arm_thickness" value="0.02"/>
-  <xacro:property name="frame_ring_radius" value="${wheel_radial_distance + wheel_width/2 + arm_length}"/>
+  <xacro:property name="frame_ring_radius" value="0.565"/> <!-- 1.13m / 2 -->
+  <xacro:property name="frame_size" value="1.13"/>
   <xacro:property name="frame_height" value="0.02"/>
   <xacro:property name="base_mass" value="3.0"/>
-  <!-- Angles for X formation (45°, 135°, 225°, 315°) -->
-  <xacro:property name="angle_ne" value="${pi/4}"/>      <!-- 45° - Northeast -->
-  <xacro:property name="angle_nw" value="${3*pi/4}"/>    <!-- 135° - Northwest -->
-  <xacro:property name="angle_sw" value="${5*pi/4}"/>    <!-- 225° - Southwest -->
-  <xacro:property name="angle_se" value="${7*pi/4}"/>    <!-- 315° - Southeast -->
+  <!-- Angles for N, W, S, E formation (0, 90, 180, 270 degrees) -->
+  <xacro:property name="angle_n" value="${0}"/>           <!-- 0° - North (+X) -->
+  <xacro:property name="angle_w" value="${pi/2}"/>        <!-- 90° - West (+Y) -->
+  <xacro:property name="angle_s" value="${pi}"/>          <!-- 180° - South (-X) -->
+  <xacro:property name="angle_e" value="${3*pi/2}"/>      <!-- 270° - East (-Y) -->
   <!-- Include materials -->
   <xacro:include filename="$(find climber_base)/urdf/materials.xacro"/>
@@ -174,17 +175,15 @@
   </xacro:macro>
   <!-- Create 4 climbing wheel assemblies in X formation -->
-  <xacro:climbing_wheel_assembly prefix="ne" angle="${angle_ne}"/>
-  <xacro:climbing_wheel_assembly prefix="nw" angle="${angle_nw}"/>
-  <xacro:climbing_wheel_assembly prefix="sw" angle="${angle_sw}"/>
-  <xacro:climbing_wheel_assembly prefix="se" angle="${angle_se}"/>
-  <!-- Connecting arcs between adjacent frame nodes (ring segments) -->
-  <xacro:macro name="frame_arc" params="name angle1 angle2">
-    <xacro:property name="mid_angle" value="${(angle1 + angle2) / 2}"/>
-    <xacro:property name="arc_len" value="${frame_ring_radius * 2 * sin((angle2 - angle1)/2)}"/>
+  <xacro:climbing_wheel_assembly prefix="n" angle="${angle_n}"/>
+  <xacro:climbing_wheel_assembly prefix="w" angle="${angle_w}"/>
+  <xacro:climbing_wheel_assembly prefix="s" angle="${angle_s}"/>
+  <xacro:climbing_wheel_assembly prefix="e" angle="${angle_e}"/>
+  <!-- Frame sides forming a square -->
+  <xacro:macro name="frame_side" params="name angle">
     <joint name="${name}_joint" type="fixed">
       <parent link="base_link"/>
       <child link="${name}"/>
-      <origin xyz="${frame_ring_radius * cos(mid_angle)} ${frame_ring_radius * sin(mid_angle)} 0"
-              rpy="0 0 ${mid_angle}"/>
+      <origin xyz="${frame_ring_radius * cos(angle)} ${frame_ring_radius * sin(angle)} 0"
+              rpy="0 0 ${angle}"/>
     </joint>
     <link name="${name}">
@@ -192,14 +191,26 @@
         <origin xyz="0 0 0" rpy="0 0 0"/>
         <geometry>
-          <box size="${arm_thickness} ${arc_len} ${arm_thickness}"/>
+          <!-- Box: thick in X (radial), long in Y (tangential), thick in Z -->
+          <box size="${arm_thickness} ${frame_size} ${arm_thickness}"/>
         </geometry>
         <material name="blue"/>
       </visual>
-    </link>
-  </xacro:macro>
-  <!-- Connect adjacent frame nodes to form the outer ring -->
-  <xacro:frame_arc name="arc_ne_nw" angle1="${angle_ne}" angle2="${angle_nw}"/>
-  <xacro:frame_arc name="arc_nw_sw" angle1="${angle_nw}" angle2="${angle_sw}"/>
-  <xacro:frame_arc name="arc_sw_se" angle1="${angle_sw}" angle2="${angle_se}"/>
-  <xacro:frame_arc name="arc_se_ne" angle1="${angle_se}" angle2="${angle_ne + 2*pi}"/>
+      <collision>
+        <origin xyz="0 0 0" rpy="0 0 0"/>
+        <geometry>
+          <box size="${arm_thickness} ${frame_size} ${arm_thickness}"/>
+        </geometry>
+      </collision>
+      <inertial>
+        <origin xyz="0 0 0" rpy="0 0 0"/>
+        <mass value="0.5"/>
+        <xacro:box_inertia m="0.5" x="${arm_thickness}" y="${frame_size}" z="${arm_thickness}"/>
+      </inertial>
+    </link>
+  </xacro:macro>
+  <!-- The 4 sides of the 113cm square frame aligned with N, W, S, E anchors -->
+  <xacro:frame_side name="frame_n" angle="${angle_n}"/>
+  <xacro:frame_side name="frame_w" angle="${angle_w}"/>
+  <xacro:frame_side name="frame_s" angle="${angle_s}"/>
+  <xacro:frame_side name="frame_e" angle="${angle_e}"/>
 </robot>

File: src/climber_base/urdf/gazebo.xacro (robot description, xacro)
@@ -6,5 +6,5 @@
   </gazebo>
   <!-- Wheel surface properties -->
-  <gazebo reference="ne_wheel">
+  <gazebo reference="n_wheel">
     <material>Gazebo/DarkGrey</material>
     <mu1>0.8</mu1>
@@ -14,5 +14,5 @@
     <minDepth>0.001</minDepth>
   </gazebo>
-  <gazebo reference="nw_wheel">
+  <gazebo reference="w_wheel">
     <material>Gazebo/DarkGrey</material>
     <mu1>0.8</mu1>
@@ -22,5 +22,5 @@
     <minDepth>0.001</minDepth>
   </gazebo>
-  <gazebo reference="sw_wheel">
+  <gazebo reference="s_wheel">
     <material>Gazebo/DarkGrey</material>
     <mu1>0.8</mu1>
@@ -30,5 +30,5 @@
     <minDepth>0.001</minDepth>
   </gazebo>
-  <gazebo reference="se_wheel">
+  <gazebo reference="e_wheel">
     <material>Gazebo/DarkGrey</material>
     <mu1>0.8</mu1>

File: src/climber_base/urdf/ros2_control.xacro (robot description, xacro)
@@ -15,5 +15,5 @@
       </xacro:unless>
       <!-- NE Wheel (Northeast - 45°) -->
-      <joint name="ne_wheel_joint">
+      <joint name="n_wheel_joint">
         <command_interface name="velocity">
           <param name="min">-10</param>
@@ -24,5 +24,5 @@
       </joint>
       <!-- NW Wheel (Northwest - 135°) -->
-      <joint name="nw_wheel_joint">
+      <joint name="w_wheel_joint">
         <command_interface name="velocity">
           <param name="min">-10</param>
@@ -33,5 +33,5 @@
       </joint>
       <!-- SW Wheel (Southwest - 225°) -->
-      <joint name="sw_wheel_joint">
+      <joint name="s_wheel_joint">
         <command_interface name="velocity">
           <param name="min">-10</param>
@@ -42,5 +42,5 @@
       </joint>
       <!-- SE Wheel (Southeast - 315°) -->
-      <joint name="se_wheel_joint">
+      <joint name="e_wheel_joint">
         <command_interface name="velocity">
           <param name="min">-10</param>
@@ -52,8 +52,8 @@
       <!-- Linear Actuators (prismatic - control wheel radial distance) -->
       <!-- NE Actuator -->
-      <joint name="ne_actuator_joint">
+      <joint name="n_actuator_joint">
         <command_interface name="position">
           <param name="min">-0.01</param>
-          <param name="max">0.04</param>
+          <param name="max">0.15</param>
         </command_interface>
         <state_interface name="position"/>
@@ -61,8 +61,8 @@
       </joint>
       <!-- NW Actuator -->
-      <joint name="nw_actuator_joint">
+      <joint name="w_actuator_joint">
         <command_interface name="position">
           <param name="min">-0.01</param>
-          <param name="max">0.04</param>
+          <param name="max">0.15</param>
         </command_interface>
         <state_interface name="position"/>
@@ -70,8 +70,8 @@
       </joint>
       <!-- SW Actuator -->
-      <joint name="sw_actuator_joint">
+      <joint name="s_actuator_joint">
         <command_interface name="position">
           <param name="min">-0.01</param>
-          <param name="max">0.04</param>
+          <param name="max">0.15</param>
         </command_interface>
         <state_interface name="position"/>
@@ -79,8 +79,8 @@
       </joint>
       <!-- SE Actuator -->
-      <joint name="se_actuator_joint">
+      <joint name="e_actuator_joint">
         <command_interface name="position">
           <param name="min">-0.01</param>
-          <param name="max">0.04</param>
+          <param name="max">0.15</param>
         </command_interface>
         <state_interface name="position"/>
