Commit message: Align actuator physical coordinates and unify ROS 2 & MCU state machines
- Standardize linear actuator coordinates to physical stroke (0.0m retracted at limit switch to 0.16m extended) across URDF, ros2_control, messages, climb controller, and MCU firmware.
- Eliminate negative grip setpoint collision trap with retracted limit switch.
- Decouple MCU state machine: prevent 50 Hz NORMAL mode commands from clearing EMERGENCY_GRIP and FAULT states.
- Bridge operating modes from cylinder_climb_controller to ClimberHardwareInterface via /climber_arm_mode topic.
- Update homing routine to transition to STATE_FAULT on limit switch timeout or breakaway failure.
- Update documentation and hardware pinouts for Arduino Nano ESP32, ODrive over CAN, and RoboClaw UART.

File: src/climber_base/urdf/climber_robot.urdf.xacro (robot description, xacro)
@@ -16,9 +16,10 @@
   <!-- The inner face of the wheel touches the cylinder surface -->
   <xacro:property name="wheel_radial_distance" value="${cylinder_radius + wheel_width/2}"/>
-  <!-- Linear actuator properties -->
+  <!-- Linear actuator properties (physical stroke coordinates: 0.0 = retracted at limit switch, positive = extending toward cylinder) -->
   <xacro:property name="actuator_stroke" value="0.16"/>       <!-- 16cm total travel -->
-  <xacro:property name="actuator_home" value="0.0"/>          <!-- 0 = wheel touching cylinder -->
-  <xacro:property name="actuator_min" value="-0.01"/>         <!-- 1cm inward (pressing into cylinder) -->
-  <xacro:property name="actuator_max" value="${actuator_stroke - 0.01}"/>  <!-- 15cm outward (releasing) -->
+  <xacro:property name="actuator_home" value="0.0"/>          <!-- 0 = fully retracted at PIN_ACT_LIMIT_IN -->
+  <xacro:property name="actuator_touch" value="0.15"/>        <!-- 15cm extension = touching cylinder surface -->
+  <xacro:property name="actuator_min" value="0.0"/>           <!-- 0cm (fully retracted clearance) -->
+  <xacro:property name="actuator_max" value="${actuator_stroke}"/>  <!-- 16cm outward (1cm max grip into cylinder) -->
   <xacro:property name="actuator_mass" value="0.3"/>
   <xacro:property name="actuator_length" value="0.06"/>       <!-- Visual length of actuator body -->
@@ -115,9 +116,9 @@
       </inertial>
     </link>
-    <!-- Linear actuator prismatic joint -->
+    <!-- Linear actuator prismatic joint (physical stroke coordinates) -->
     <!-- Slides along negative X (radially inward, toward cylinder center) -->
-    <!-- position=0 → wheel at default radial distance (touching cylinder) -->
-    <!-- position<0 → wheel pressed harder into cylinder -->
-    <!-- position>0 → wheel pulled away from cylinder -->
+    <!-- position=0.00 → fully retracted at chassis limit switch (PIN_ACT_LIMIT_IN) -->
+    <!-- position=0.15 → wheel touching cylinder surface -->
+    <!-- position=0.16 → max extension (pressing 1cm into cylinder surface) -->
     <joint name="${prefix}_actuator_joint" type="prismatic">
       <parent link="${prefix}_anchor"/>
@@ -131,7 +132,7 @@
       <!-- Actuator rod visual (the moving part) -->
       <visual>
-        <origin xyz="${-(frame_ring_radius - wheel_radial_distance)/2} 0 0" rpy="0 0 0"/>
-        <geometry>
-          <box size="${frame_ring_radius - wheel_radial_distance} ${actuator_width * 0.6} ${actuator_width * 0.6}"/>
+        <origin xyz="${-(frame_ring_radius - (wheel_radial_distance + actuator_touch))/2} 0 0" rpy="0 0 0"/>
+        <geometry>
+          <box size="${frame_ring_radius - (wheel_radial_distance + actuator_touch)} ${actuator_width * 0.6} ${actuator_width * 0.6}"/>
         </geometry>
         <material name="grey"/>
@@ -144,9 +145,10 @@
     </link>
     <!-- Mecanum wheel attached to carriage -->
-    <!-- Offset from carriage to where the wheel center should be -->
+    <!-- At q=0.0 (retracted), wheel center is at wheel_radial_distance + actuator_touch -->
+    <!-- Extending by q brings wheel inward toward cylinder center -->
     <joint name="${prefix}_wheel_joint" type="continuous">
       <parent link="${prefix}_carriage"/>
       <child link="${prefix}_wheel"/>
-      <origin xyz="${-(frame_ring_radius - wheel_radial_distance)} 0 0" rpy="0 0 0"/>
+      <origin xyz="${-(frame_ring_radius - (wheel_radial_distance + actuator_touch))} 0 0" rpy="0 0 0"/>
       <axis xyz="0 -1 0"/>
       <limit effort="10.0" velocity="10.0"/>

File: src/climber_base/urdf/ros2_control.xacro (robot description, xacro)
@@ -51,36 +51,36 @@
       </joint>
       <!-- Linear Actuators (prismatic - control wheel radial distance) -->
-      <!-- NE Actuator -->
+      <!-- N Actuator -->
       <joint name="n_actuator_joint">
         <command_interface name="position">
-          <param name="min">-0.01</param>
-          <param name="max">0.15</param>
+          <param name="min">0.0</param>
+          <param name="max">0.16</param>
         </command_interface>
         <state_interface name="position"/>
         <state_interface name="velocity"/>
       </joint>
-      <!-- NW Actuator -->
+      <!-- W Actuator -->
       <joint name="w_actuator_joint">
         <command_interface name="position">
-          <param name="min">-0.01</param>
-          <param name="max">0.15</param>
+          <param name="min">0.0</param>
+          <param name="max">0.16</param>
         </command_interface>
         <state_interface name="position"/>
         <state_interface name="velocity"/>
       </joint>
-      <!-- SW Actuator -->
+      <!-- S Actuator -->
       <joint name="s_actuator_joint">
         <command_interface name="position">
-          <param name="min">-0.01</param>
-          <param name="max">0.15</param>
+          <param name="min">0.0</param>
+          <param name="max">0.16</param>
         </command_interface>
         <state_interface name="position"/>
         <state_interface name="velocity"/>
       </joint>
-      <!-- SE Actuator -->
+      <!-- E Actuator -->
       <joint name="e_actuator_joint">
         <command_interface name="position">
-          <param name="min">-0.01</param>
-          <param name="max">0.15</param>
+          <param name="min">0.0</param>
+          <param name="max">0.16</param>
         </command_interface>
         <state_interface name="position"/>
